File: amp-brd-v2/opamp.kicad_sch (KiCad schematic)
At the start: 17 parts, among them U1 OPA547F, U2 INA233

Commit message: Added FB smoothing capacitor to amp brd
Parts:
- removed U1: OPA547F, project_footprints:KTW0007A, symbol project_symbols:OPA547F
- added C6: 0.01u, Capacitor_SMD:C_0805_2012Metric, symbol Device:C
- added U1: OPA548, project_footprints:KTW0007A, symbol project_symbols:OPA548
- A00, A01: value SolderJumper_3_Open -> L / NC / R
- A10, A11: value SolderJumper_3_Open -> NC
Connections:
- net CTRL_{IN}: now also U1.1 (+)
- net GND: now also U1.4 (V-), U1.8 (EP)
- net ILIM: now also U1.3 (I_{LIM})
- net OP_FB: now also C6.2, U1.2 (-)
- net PWRIN: now also U1.5 (V+)
- net STAT_PIN: now also U1.7 (~{DIS})
- net V_{RAW}: now also C6.1, U1.6

Commit message: Modified DAC, AMP v2 and Mezzanine to support AMP v3. Finished AMP v3 design.
Parts:
- R1: value 10k -> 13k; Mfr Walsin -> TE Connectivity / Holsworthy; Mfr # WF08P1002FTL -> CRG0805F13K; Mouser # 791-WF08P1002FTL -> 279-CRG0805F13K; Mouser URL https://www.mouser.com/ProductDetail/Walsin/WF08P1002FTL?qs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 -> https://www.mouser.com/ProductDetail/TE-Connectivity-Holswo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
Changed lines of the file:
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@@
 			)
 		)
-		(property "Value" "10k"
+		(property "Value" "13k"
 			(at 119.38 146.05 90)
 			(effects
@@
 			)
 		)
-		(property "Datasheet" "https://www.mouser.com/datasheet/3/317/1/ASC_WFxxP.pdf"
+		(property "Datasheet" "https://www.te.com/commerce/DocumentDelivery/DDEController?Action=srchrtrv&DocNm=1623112&DocType=Customer+Drawing&DocLang=English&PartCntxt=1623112-1"
 			(at 119.38 146.05 0)
 			(effects
@@
 			)
 		)
-		(property "Description" "Thin Film Resistors 10K Ohms 250mW +/- 1% 0805"
+		(property "Description" "Thick Film Resistors CRG0805 1% 13K"
 			(at 119.38 146.05 0)
 			(effects
@@
 			)
 		)
-		(property "Mfr" "Walsin"
+		(property "Mfr" "TE Connectivity / Holsworthy "
 			(at 119.38 146.05 90)
 			(effects
@@
 			)
 		)
-		(property "Mfr #" "WF08P1002FTL"
+		(property "Mfr #" "CRG0805F13K"
 			(at 119.38 146.05 90)
 			(effects
@@
 			)
 		)
-		(property "Mouser #" "791-WF08P1002FTL"
+		(property "Mouser #" "279-CRG0805F13K"
 			(at 119.38 146.05 90)
 			(effects
@@
 			)
 		)
-		(property "Mouser URL" "https://www.mouser.com/ProductDetail/Walsin/WF08P1002FTL?qs=sGAEpiMZZMvdGkrng054t7z4BkURc4LzCx%252B5OuE3qppREPl7ULZTTA%3D%3D"
+		(property "Mouser URL" "https://www.mouser.com/ProductDetail/TE-Connectivity-Holsworthy/CRG0805F13K?qs=sGAEpiMZZMvdGkrng054t%252BGQy31YLTNMxyRamAR5vSg%3D"
 			(at 119.38 146.05 90)
 			(effects
