File: amp-brd-v3/opamp.kicad_sch (KiCad schematic)
At the start: 18 parts, among them U2 INA233, U4 LMR36510ADDA

Commit message: Final review with Joe
Parts:
- added D2, D3: D_Schottky, Diode_SMD:D_0402_1005Metric, symbol Device:D_Schottky
- added R4: 0, Resistor_SMD:R_0402_1005Metric, symbol Device:R
Connections:
- net CTRL_{IN}: now also D3.2 (A), R4.1; no longer R2.2, R3.2
- net GND: now also D2.2 (A)
- new net FCTRL: D2.1 (K), D3.1 (K), R2.2, R3.2, R4.2
