File: amp-brd-v4/amp-brd-v4.kicad_sch (KiCad schematic)
At the start: 1 part, among them U1 MCP19061

Commit message: Added MCP19061 calculator
Parts:
- added C1, C2, C3, C4: 4.7u, Capacitor_SMD:C_0805_2012Metric, symbol Device:C
- added C5: 1u, Capacitor_SMD:C_0603_1608Metric, symbol Device:C
- added C6: 1u, Capacitor_SMD:C_0805_2012Metric, symbol Device:C
- added R1, R2: 10k, Resistor_SMD:R_0402_1005Metric, symbol Device:R
- added R3, R4: 5m, Resistor_SMD:R_0402_1005Metric, symbol Device:R
Connections:
- net GND_{A} is gone; now on net GND: U1.10 (GND_{D}), U1.12 (GND_{A}), U1.15 (NC), U1.16 (NC), U1.23 (GND_{P}), U1.EP (GND)
- net ~{SHDN}: now reaches U1.1 (~{SHDN})
- net EN: now reaches U1.2 (EN)
- net GND: now reaches U1.3 (ADDR)
- net GND: now also U1.30 (V_{OUT}-), C1.2, C2.2, C3.2, C4.2, C5.2, C6.2
- net SCL: now reaches U1.4 (SCL)
- net SCL: now also R2.2
- net SDA: now reaches U1.5 (SDA)
- net SDA: now also R1.2
- net ~{ALRT}: now reaches U1.6 (~{ALRT})
- net +3V3: now reaches U1.8 (VDD_{IO})
- net +3V3: now also C5.1, R1.1, R2.1
- net at U1.11 (ADC_{REF}): now also C4.1
- net at U1.13 (AV_{DD}): now also C2.1
- net at U1.25 (V_{DD}): now also C1.1
- net at U1.9 (DV_{DD}): now also C3.1
- net VIN_S: now reaches U1.14 (V_{IN})
- net VIN_S: now also U1.18 (I_{IN}-), R3.2
- net VIN: now reaches U1.17 (I_{IN}+)
- net VIN: now also C6.1, R3.1
- net VOUT_S: now reaches U1.29 (V_{OUT}+)
- net VOUT_S: now also U1.32 (I_{OUT}+), R4.1
- net VOUT: now reaches U1.31 (I_{OUT}-)
- net VOUT: now also R4.2
- no-connect marks 0 -> 1
Other:
- moved on the sheet: U1A, U1B, U1C
